Commit message: Migrate to xArm6 and improve face tracking and recovery
- Make xArm6 the default robot while retaining Lite 6 support
- Check robot identity and joint limits before hardware activation
- Prioritize face alignment and improve recovery from constrained poses
- Add Kalman and One Euro filters for the tracked face position
- Expand runtime camera, geometry and motion configuration
- Support configuration changes without rebuilding the Docker image
- Add stress scenarios and regression tests for difficult starting poses,
  rapid target motion, close approaches and target switching
- Update hardware, Docker, camera and simulation documentation

File: description/lite6_hardware.urdf.xacro (robot description, xacro)
@@ -2,4 +2,16 @@
 <!-- Real and mock ros2_control assembly; no Gazebo tags or sensors. -->
 <robot name="lite6" xmlns:xacro="http://www.ros.org/wiki/xacro">
+  <xacro:arg name="joint1_lower_limit" default="-6.283185307179586"/>
+  <xacro:arg name="joint1_upper_limit" default="6.283185307179586"/>
+  <xacro:arg name="joint2_lower_limit" default="-2.6179938779914944"/>
+  <xacro:arg name="joint2_upper_limit" default="2.6179938779914944"/>
+  <xacro:arg name="joint3_lower_limit" default="-0.061086523819801536"/>
+  <xacro:arg name="joint3_upper_limit" default="5.235987755982989"/>
+  <xacro:arg name="joint4_lower_limit" default="-6.283185307179586"/>
+  <xacro:arg name="joint4_upper_limit" default="6.283185307179586"/>
+  <xacro:arg name="joint5_lower_limit" default="-2.1642082724729685"/>
+  <xacro:arg name="joint5_upper_limit" default="2.1642082724729685"/>
+  <xacro:arg name="joint6_lower_limit" default="-6.283185307179586"/>
+  <xacro:arg name="joint6_upper_limit" default="6.283185307179586"/>
   <xacro:arg name="config_file" default=""/>
   <xacro:arg name="camera_mode" default="mono_cpu"/>
@@ -26,4 +38,16 @@
   </joint>
   <xacro:lite6_urdf prefix=""
+    joint1_lower_limit="$(arg joint1_lower_limit)"
+    joint1_upper_limit="$(arg joint1_upper_limit)"
+    joint2_lower_limit="$(arg joint2_lower_limit)"
+    joint2_upper_limit="$(arg joint2_upper_limit)"
+    joint3_lower_limit="$(arg joint3_lower_limit)"
+    joint3_upper_limit="$(arg joint3_upper_limit)"
+    joint4_lower_limit="$(arg joint4_lower_limit)"
+    joint4_upper_limit="$(arg joint4_upper_limit)"
+    joint5_lower_limit="$(arg joint5_lower_limit)"
+    joint5_upper_limit="$(arg joint5_upper_limit)"
+    joint6_lower_limit="$(arg joint6_lower_limit)"
+    joint6_upper_limit="$(arg joint6_upper_limit)"
     kinematics_params_filename="$(find face_tracking_arm)/description/ufactory_lite6/config/kinematics/default/lite6_default_kinematics.yaml"/>
   <xacro:monitor_model parent="link6" thickness="${monitor['size_m'][0]}"
@@ -60,8 +84,28 @@
     </xacro:if>
   </xacro:if>
+  <xacro:unless value="${mount['publish_optical_tf']}">
+    <link name="tracking_gaze_optical"/>
+    <joint name="tracking_gaze_joint" type="fixed">
+      <parent link="${mount['body_frame']}"/><child link="tracking_gaze_optical"/>
+      <origin xyz="${' '.join(map(str, cameras['left']['optical_xyz_m']))}"
+        rpy="${' '.join([str(v * degree_scale) for v in cameras['left']['optical_rpy_deg']])}"/>
+    </joint>
+  </xacro:unless>
   <xacro:unless value="$(arg mock_hardware)">
     <!-- Use the manufacturer's interface declaration and actual bounded joints. -->
     <xacro:include filename="$(find xarm_description)/urdf/lite6/lite6.ros2_control.xacro"/>
     <xacro:lite6_ros2_control prefix="" hw_ns="ufactory" robot_ip="${hardware['robot']['ip']}"
+      joint1_lower_limit="$(arg joint1_lower_limit)"
+    joint1_upper_limit="$(arg joint1_upper_limit)"
+    joint2_lower_limit="$(arg joint2_lower_limit)"
+    joint2_upper_limit="$(arg joint2_upper_limit)"
+    joint3_lower_limit="$(arg joint3_lower_limit)"
+    joint3_upper_limit="$(arg joint3_upper_limit)"
+    joint4_lower_limit="$(arg joint4_lower_limit)"
+    joint4_upper_limit="$(arg joint4_upper_limit)"
+    joint5_lower_limit="$(arg joint5_lower_limit)"
+    joint5_upper_limit="$(arg joint5_upper_limit)"
+    joint6_lower_limit="$(arg joint6_lower_limit)"
+    joint6_upper_limit="$(arg joint6_upper_limit)"
       report_type="${hardware['robot']['report_type']}" add_gripper="false" velocity_control="false"/>
   </xacro:unless>

File: description/lite6_table.urdf.xacro (robot description, xacro)
@@ -24,5 +24,5 @@
   <xacro:arg
     name="initial_positions_file"
-    default="$(find face_tracking_arm)/config/control/initial_positions.yaml"/>
+    default="$(find face_tracking_arm)/config/control/lite6_initial_positions.yaml"/>
   <xacro:arg
     name="controller_config_file"

File: description/monitor.urdf.xacro (robot description, xacro)
@@ -1,10 +1,10 @@
 <?xml version="1.0"?>
 <!--
-  Responsibility: define the simulated display attached to the Lite 6 flange
+  Responsibility: define the display attached to the robot flange
   and expose the center of its front surface as the control frame.
 -->
 <robot xmlns:xacro="http://www.ros.org/wiki/xacro">
-  <xacro:macro name="monitor_model" params="parent prefix:='' thickness:=0.03 width:=0.30
-    height:=0.20 mass:=0.50 mount_xyz:='' mount_rpy:='${pi} ${-pi / 2.0} 0'">
+  <xacro:macro name="monitor_model" params="parent prefix:='' thickness:=0.010 width:=0.355
+    height:=0.224 mass:=0.692 mount_xyz:='' mount_rpy:='${pi} ${-pi / 2.0} 0'">
     <!-- Local axes: +X points out of the screen, +Y spans its width, +Z its height. -->
     <xacro:property name="monitor_thickness" value="${thickness}"/>
@@ -22,30 +22,33 @@
       value="${monitor_mass * (monitor_thickness * monitor_thickness + monitor_width * monitor_width) / 12.0}"/>
     <link name="${prefix}monitor_link">
-      <inertial>
-        <origin xyz="0 0 0" rpy="0 0 0"/>
-        <mass value="${monitor_mass}"/>
-        <inertia
-          ixx="${monitor_ixx}"
-          ixy="0"
-          ixz="0"
-          iyy="${monitor_iyy}"
-          iyz="0"
-          izz="${monitor_izz}"/>
-      </inertial>
-      <visual name="${prefix}monitor_visual">
-        <origin xyz="0 0 0" rpy="0 0 0"/>
-        <geometry>
-          <box size="${monitor_thickness} ${monitor_width} ${monitor_height}"/>
-        </geometry>
-        <material name="${prefix}monitor_dark">
-          <color rgba="0.08 0.08 0.10 1.0"/>
-        </material>
-      </visual>
-      <collision name="${prefix}monitor_collision">
-        <origin xyz="0 0 0" rpy="0 0 0"/>
-        <geometry>
-          <box size="${monitor_thickness} ${monitor_width} ${monitor_height}"/>
-        </geometry>
-      </collision>
+      <!-- All-zero dimensions retain the mount/TF chain without a physical box. -->
+      <xacro:unless value="${monitor_thickness == 0 and monitor_width == 0 and monitor_height == 0}">
+        <inertial>
+          <origin xyz="0 0 0" rpy="0 0 0"/>
+          <mass value="${monitor_mass}"/>
+          <inertia
+            ixx="${monitor_ixx}"
+            ixy="0"
+            ixz="0"
+            iyy="${monitor_iyy}"
+            iyz="0"
+            izz="${monitor_izz}"/>
+        </inertial>
+        <visual name="${prefix}monitor_visual">
+          <origin xyz="0 0 0" rpy="0 0 0"/>
+          <geometry>
+            <box size="${monitor_thickness} ${monitor_width} ${monitor_height}"/>
+          </geometry>
+          <material name="${prefix}monitor_dark">
+            <color rgba="0.08 0.08 0.10 1.0"/>
+          </material>
+        </visual>
+        <collision name="${prefix}monitor_collision">
+          <origin xyz="0 0 0" rpy="0 0 0"/>
+          <geometry>
+            <box size="${monitor_thickness} ${monitor_width} ${monitor_height}"/>
+          </geometry>
+        </collision>
+      </xacro:unless>
     </link>
     <!--

File: description/monitor_cameras.urdf.xacro (robot description, xacro)
@@ -6,5 +6,5 @@
     <joint name="${name}_mount" type="fixed">
       <parent link="monitor_camera_bar"/><child link="${name}_frame"/>
-      <origin xyz="0.018 ${lateral} 0"/>
+      <origin xyz="${camera_depth / 2 + .001} ${lateral} 0"/>
     </joint>
     <link name="${frame}"/>
@@ -15,10 +15,10 @@
     <gazebo reference="monitor_camera_bar">
       <sensor name="${name}" type="camera">
-        <pose>0.018 ${lateral} 0 0 0 0</pose>
-        <always_on>true</always_on><update_rate>30</update_rate>
+        <pose>${camera_depth / 2 + .001} ${lateral} 0 0 0 0</pose>
+        <always_on>true</always_on><update_rate>${camera_rate}</update_rate>
         <topic>${topic}</topic>
         <camera>
-          <horizontal_fov>${pi / 3}</horizontal_fov>
-          <image><width>640</width><height>480</height><format>R8G8B8</format></image>
+          <horizontal_fov>${horizontal_fov}</horizontal_fov>
+          <image><width>${image_width}</width><height>${image_height}</height><format>R8G8B8</format></image>
           <clip><near>0.05</near><far>20</far></clip>
           <camera_info_topic>${info}</camera_info_topic>
@@ -26,9 +26,9 @@
           <lens>
             <intrinsics>
-              <fx>${camera_focal}</fx><fy>${camera_focal}</fy><cx>320</cx><cy>240</cy><s>0</s>
+              <fx>${camera_focal}</fx><fy>${camera_focal}</fy><cx>${image_width / 2}</cx><cy>${image_height / 2}</cy><s>0</s>
             </intrinsics>
             <projection>
               <p_fx>${camera_focal}</p_fx><p_fy>${camera_focal}</p_fy>
-              <p_cx>320</p_cx><p_cy>240</p_cy><tx>${tx}</tx><ty>0</ty>
+              <p_cx>${image_width / 2}</p_cx><p_cy>${image_height / 2}</p_cy><tx>${tx}</tx><ty>0</ty>
             </projection>
           </lens>
@@ -37,23 +37,24 @@
     </gazebo>
   </xacro:macro>
-  <xacro:macro name="monitor_cameras" params="mode baseline">
-    <xacro:property name="camera_focal" value="554.2562584220407"/>
+  <xacro:macro name="monitor_cameras" params="mode baseline horizontal_fov:=1.433 image_width:=1280 image_height:=720
+    camera_rate:=30 monitor_height:=0.224 camera_depth:=0.027 camera_height:=0.0265">
+    <xacro:property name="camera_focal" value="${image_width / (2 * tan(horizontal_fov / 2))}"/>
     <xacro:property name="stereo" value="${mode == 'stereo'}"/>
-    <xacro:property name="bar_width" value="${baseline + 0.028 if stereo else 0.04}"/>
-    <xacro:property name="bar_mass" value="0.03"/>
+    <xacro:property name="bar_width" value="${max(0.102, baseline + 0.028) if stereo else 0.102}"/>
+    <xacro:property name="bar_mass" value="0.065"/>
     <link name="monitor_camera_bar">
       <inertial>
         <mass value="${bar_mass}"/>
-        <inertia ixx="${bar_mass * (bar_width**2 + 0.028**2) / 12}" ixy="0" ixz="0"
-          iyy="${bar_mass * (0.034**2 + 0.028**2) / 12}" iyz="0"
-          izz="${bar_mass * (0.034**2 + bar_width**2) / 12}"/>
+        <inertia ixx="${bar_mass * (bar_width**2 + camera_height**2) / 12}" ixy="0" ixz="0"
+          iyy="${bar_mass * (camera_depth**2 + camera_height**2) / 12}" iyz="0"
+          izz="${bar_mass * (camera_depth**2 + bar_width**2) / 12}"/>
       </inertial>
       <visual>
-        <geometry><box size="0.034 ${bar_width} 0.028"/></geometry>
+        <geometry><box size="${camera_depth} ${bar_width} ${camera_height}"/></geometry>
         <material name="camera_dark"><color rgba="0.04 0.04 0.05 1"/></material>
       </visual>
-      <collision><geometry><box size="0.036 ${bar_width} 0.028"/></geometry></collision>
+      <collision><geometry><box size="${camera_depth} ${bar_width} ${camera_height}"/></geometry></collision>
       <visual name="left_lens">
-        <origin xyz="0.017 ${baseline / 2 if stereo else 0} 0" rpy="0 ${pi / 2} 0"/>
+        <origin xyz="${camera_depth / 2} ${baseline / 2 if stereo else 0} 0" rpy="0 ${pi / 2} 0"/>
         <geometry><cylinder radius="0.008" length="0.002"/></geometry>
         <material name="camera_glass"><color rgba="0.1 0.35 0.6 1"/></material>
@@ -61,5 +62,5 @@
       <xacro:if value="${stereo}">
         <visual name="right_lens">
-          <origin xyz="0.017 ${-baseline / 2} 0" rpy="0 ${pi / 2} 0"/>
+          <origin xyz="${camera_depth / 2} ${-baseline / 2} 0" rpy="0 ${pi / 2} 0"/>
           <geometry><cylinder radius="0.008" length="0.002"/></geometry>
           <material name="camera_glass"/>
@@ -69,5 +70,5 @@
     <joint name="monitor_camera_mount" type="fixed">
       <parent link="monitor_link"/><child link="monitor_camera_bar"/>
-      <origin xyz="0 0 0.114"/>
+      <origin xyz="0 0 ${monitor_height / 2 + camera_height / 2}"/>
     </joint>
     <xacro:monitor_rgb_sensor name="monitor_left_camera"

Commit message: Add camera mount calibration and RGB-D hardware support

File: description/lite6_hardware.urdf.xacro (robot description, xacro)
@@ -66,5 +66,5 @@
   </link>
   <joint name="hardware_camera_mount" type="fixed">
-    <parent link="monitor_link"/><child link="${mount['body_frame']}"/>
+    <parent link="link6"/><child link="${mount['body_frame']}"/>
     <origin xyz="${' '.join(map(str, mount['xyz_m']))}"
       rpy="${' '.join([str(v * degree_scale) for v in mount['rpy_deg']])}"/>

File: description/xarm6_hardware.urdf.xacro (robot description, xacro)
@@ -67,5 +67,5 @@
   </link>
   <joint name="hardware_camera_mount" type="fixed">
-    <parent link="monitor_link"/><child link="${mount['body_frame']}"/>
+    <parent link="link6"/><child link="${mount['body_frame']}"/>
     <origin xyz="${' '.join(map(str, mount['xyz_m']))}"
       rpy="${' '.join([str(v * degree_scale) for v in mount['rpy_deg']])}"/>
